Commit message: working pybullet application

File: RoboticArm_Simulation_Software/example.urdf (robot description, URDF)
Before this commit: robot six_dof_robot, 7 links, 6 joints
Links:
- added link end_effector, mass 0.3; visual box size=0.1 0.1 0.1
- link base_link: mass None -> 1.0; geometry visual cylinder length=0.3 radius=0.2
- link link_1: mass None -> 1.0; geometry visual cylinder length=0.5 radius=0.15
- link link_2: mass None -> 1.0; geometry visual cylinder length=0.6 radius=0.12
- link link_3: mass None -> 1.0; geometry visual cylinder length=0.7 radius=0.1
- link link_4: mass None -> 0.5; geometry visual cylinder length=0.2 radius=0.09
- link link_5: mass None -> 0.5; geometry visual cylinder length=0.2 radius=0.08
- link link_6: mass None -> 0.5; geometry visual cylinder length=0.15 radius=0.07
Joints:
- added joint joint_7: type fixed, parent link_6, child end_effector, origin xyz=0 0 0.15 rpy=0 0 0
- joint joint_1: limit lower=-1.57 upper=1.57 effort=100 velocity=1.0 -> lower=-3.14 upper=3.14 effort=100 velocity=1; origin xyz=0 0 0.1 rpy=0 0 0 -> xyz=0 0 0.15 rpy=0 0 0
- joint joint_2: limit lower=-1.57 upper=1.57 effort=100 velocity=1.0 -> lower=-3.14 upper=3.14 effort=100 velocity=1; origin xyz=0 0 0.3 rpy=0 0 0 -> xyz=0 0 0.5 rpy=0 1.57 0
- joint joint_3: limit lower=-1.57 upper=1.57 effort=100 velocity=1.0 -> lower=-3.14 upper=3.14 effort=100 velocity=1; origin xyz=0 0 0.3 rpy=0 0 0 -> xyz=0 0 0.6 rpy=0 0 0
- joint joint_4: limit lower=-1.57 upper=1.57 effort=100 velocity=1.0 -> lower=-3.14 upper=3.14 effort=100 velocity=1; origin xyz=0 0 0.3 rpy=0 0 0 -> xyz=0 0 0.7 rpy=0 1.57 0
- joint joint_5: axis 0 1 0 -> 0 0 1; limit lower=-1.57 upper=1.57 effort=100 velocity=1.0 -> lower=-3.14 upper=3.14 effort=100 velocity=1; origin xyz=0 0 0.3 rpy=0 0 0 -> xyz=0 0 0.2 rpy=0 1.57 0
- joint joint_6: axis 0 1 0 -> 0 0 1; limit lower=-1.57 upper=1.57 effort=100 velocity=1.0 -> lower=-3.14 upper=3.14 effort=100 velocity=1; origin xyz=0 0 0.3 rpy=0 0 0 -> xyz=0 0 0.2 rpy=0 1.57 0
